File: hw/ev_simulator/ev_emulator.brd (EAGLE design)
At the start: 100 x 80 mm, 57 parts, among them IC1 LM324N, Q1 BC337, Q2 BC337, Q3 BC337, Q4 BC337

Commit message: Finished working prototype
Parts:
- moved R21 168.7 mm to (83.3, 54.9), turned to 90 degrees
- moved CUSTOM 164.4 mm to (86.1, 18.2)
- moved VENTELATE 152.5 mm to (86.1, 27.4)
- moved R20 151.7 mm to (75.7, 54.9), turned to 90 degrees
- moved PROX 146.1 mm to (89.7, 47.2), turned to 90 degrees
- moved R4 144.3 mm to (80.1, 28.2), turned to 270 degrees
- moved PILOT 138.4 mm to (89.7, 53.6), turned to 90 degrees
- moved R25 136.2 mm to (78.2, 54.9), turned to 270 degrees
- moved R3 129.7 mm to (80.8, 42.2), turned to 270 degrees
- moved R13 127.6 mm to (30.0, 16.8), turned to 90 degrees
- moved R2 127.5 mm to (76.0, 20.1), turned to 270 degrees
- moved LED3 126.6 mm to (31.2, 9.14), turned to 270 degrees
- moved IC1 122.9 mm to (79.5, 66.3)
- moved R7 122.8 mm to (36.3, 51.1)
- moved R28 122.2 mm to (38.3, 70.1), turned to 180 degrees
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Connections:
- removed net V+: IC1.4
- removed net V-: IC1.11
- net 3.3V: now also U$1.P$20
- net 5V: now also IC1.4, U$1.P$18
- net GND: now also CUSTOM.1, IC1.11, U$1.P$19; no longer CUSTOM.3
- net N$17: now also CUSTOM.3; no longer CUSTOM.1
Routing:
- net GND: track 0.00 -> 362.2 mm, vias 0 -> 2
- net 5V: track 0.00 -> 200.9 mm, vias 0 -> 2
- net N$28: track 0.00 -> 184.1 mm
- net N$36: track 0.00 -> 76.3 mm
- net 3.3V: track 0.00 -> 60.0 mm
- net N$3: track 0.00 -> 42.6 mm
- net N$13: track 0.00 -> 32.3 mm
- net N$5: track 0.00 -> 31.0 mm
- net N$15: track 0.00 -> 27.0 mm
- net N$20: track 0.00 -> 26.7 mm
- net N$2: track 0.00 -> 26.6 mm
- net N$17: track 0.00 -> 26.4 mm
- net N$14: track 0.00 -> 24.9 mm
- net N$32: track 0.00 -> 24.3 mm
- net N$12: track 0.00 -> 23.6 mm
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Other:
- board size 100 x 80 mm -> 100 x 80.1 mm
