File: hw/ev_simulator/ev_emulator.sch (EAGLE design)
At the start: 15 parts

Commit message: Updated hw and sw
Parts:
- removed OK1, OK2, OK3: PC817, optocoupler:PC817
- removed R1: 2000, antduino:SPARKFUN_RESISTORAXIAL-0.3
- removed R2: 680, antduino:SPARKFUN_RESISTORAXIAL-0.3
- removed U$2: AZ850, AZ850:AZ850
- added 1, 2, 3: AZ850, AZ850:AZ850
- added C1, C2, C3: 10nF, capacitor-wima:C2,5-3
- added CUSTOM, VENTELATE: switch, antduino:SPARKFUN-ELECTROMECHANICAL_SWITCH-MOMENTARY-2PTH
- added D1, D2, D3: 1N4446, diode:1N4446
- added IC1: LM324N, linear:LM324N
- added LED1, LED2, LED3: (no value), antduino:SPARKFUN_LED-3MM-NO_SILK
- added Q1, Q4, Q5: D882, transistor-npn:BF459
- added Q2: BC337, transistor-npn:BC337
- added R10, R14, R16: 22, antduino:SPARKFUN_RESISTORAXIAL-0.3
- added R11, R15, R21, R9: 100K, antduino:SPARKFUN_RESISTORAXIAL-0.3
- added R12: 4.7K, antduino:SPARKFUN_RESISTORAXIAL-0.3
- added R13, R8: 500, antduino:SPARKFUN_RESISTORAXIAL-0.3
- added R17: 330, antduino:SPARKFUN_RESISTORAXIAL-0.3
- added R18: 1.3K, antduino:SPARKFUN_RESISTORAXIAL-0.3
- added R19: 2.74K, antduino:SPARKFUN_RESISTORAXIAL-0.3
- added R20: 150, antduino:SPARKFUN_RESISTORAXIAL-0.3
- added R22: 200K, antduino:SPARKFUN_RESISTORAXIAL-0.3
- added R23, R25: 1K, antduino:SPARKFUN_RESISTORAXIAL-0.3
- added R24: 2K, antduino:SPARKFUN_RESISTORAXIAL-0.3
- R5, R7: value 330 -> 4.7K
- R6: value 330 -> 500
- U$3: value AZ850 -> DISPLAY-OLED-128X64-I2C; device AZ850:AZ850 -> diy-modules:DISPLAY-OLED-128X64-I2C
Connections:
- removed net N$1: PILOT.1, R1.2
- new net 5V: R10.1, R14.1, R16.1, R25.2
- new net N$10: LED1.A, R8.1
- new net N$11: Q4.B, R5.1, R9.2
- new net N$12: 2.С_1, C2.1, D2.A, LED2.C, Q4.C
- new net N$13: U$1.PC14, VENTELATE.1
- new net N$14: U$1.PB7, U$3.SDA
- new net N$15: U$1.PB6, U$3.SCL
- new net N$16: 2.С_2, C2.2, D2.C, R10.2, R6.2
- new net N$17: CUSTOM.1, U$1.PC13
- new net N$18: LED2.A, R6.1
- new net N$19: Q5.B, R12.1, R15.2
- new net N$20: 1.С_1, C3.1, D3.A, LED3.C, Q5.C
- new net N$21: 1.С_2, C3.2, D3.C, R13.2, R16.2
- new net N$22: LED3.A, R13.1
- new net N$23: 1.4, R17.1
- new net N$24: R23.2, R24.2, U$1.PA6
- new net N$25: 2.4, R18.1
- new net N$26: 3.4, R19.1
- new net N$27: IC1A.+IN, R21.2, R22.2
- new net N$28: PILOT.1, R17.2, R18.2, R19.2, R22.1
- new net N$29: IC1A.-IN, R20.2, R25.1
- new net N$30: IC1A.OUT, R23.1
- net 3.3V: now also U$3.VCC
- net GND: now also 1.3, 2.3, 3.3, CUSTOM.2, Q1.E, Q4.E, Q5.E, R11.1, R15.1, R20.1, R21.1, R24.1, R9.1, U$3.GND, VENTELATE.2; no longer OK1.C, OK2.C, OK3.C, R2.1
- net N$2: no longer R1.1, R2.2, U$1.PA6
- net N$4: now also Q1.B, R11.2, R7.1; no longer OK1.A, R5.1
- net N$5: now also R12.2; no longer R5.2
- net N$6: now also 3.С_1, C1.1, D1.A, LED1.C, Q1.C; no longer OK2.A, R6.1
- net N$7: now also 3.С_2, C1.2, D1.C, R14.2, R8.2; no longer OK3.A, R7.1
- net N$8: now also R5.2; no longer R6.2
Other:
- moved on the sheet: PILOT, PROX, R3, R4, R5, R6, R7

Commit message: Added changed hw
Parts:
- removed Q5: D882, transistor-npn:BF459
- added 4: AZ850, AZ850:AZ850
- added C4: 10nF, capacitor-wima:C2,5-3
- added D4, D5: 1N4446, diode:1N4446
- added LED4: (no value), antduino:SPARKFUN_LED-3MM-NO_SILK
- added Q3: BC337, transistor-npn:BC337
- added R1: 220K, antduino:SPARKFUN_RESISTORAXIAL-0.3
- added R2: 68K, antduino:SPARKFUN_RESISTORAXIAL-0.3
- added R26: 4.7K, antduino:SPARKFUN_RESISTORAXIAL-0.3
- added R27: 500, antduino:SPARKFUN_RESISTORAXIAL-0.3
- added R28: 100K, antduino:SPARKFUN_RESISTORAXIAL-0.3
- added R29: 22, antduino:SPARKFUN_RESISTORAXIAL-0.3
- Q1, Q4: value D882 -> BC337; device transistor-npn:BF459 -> transistor-npn:BC337
Connections:
- new net N$1: R26.2, U$1.PA10
- new net N$31: Q4.B, R26.1, R28.2
- new net N$32: 4.С_1, C4.1, D4.A, LED4.C, Q4.C
- new net N$33: 4.С_2, C4.2, D4.C, R27.2, R29.2
- new net N$34: LED4.A, R27.1
- new net N$36: 1.3, 2.3, 3.3, 4.4, D5.A
- net 5V: now also R29.1
- net GND: now also 4.3, D5.C, Q2.E, Q3.E, R2.2, R28.1; no longer 1.3, 2.3, 3.3, Q5.E
- net N$11: now also Q1.B; no longer Q4.B
- net N$12: now also Q1.C; no longer Q4.C
- net N$19: now also Q3.B; no longer Q5.B
- net N$2: now also R1.2, R2.1
- net N$20: now also Q3.C; no longer Q5.C
- net N$28: now also R1.1
- net N$4: now also Q2.B; no longer Q1.B
- net N$6: now also Q2.C; no longer Q1.C
Other:
- moved on the sheet: Q1, Q2, Q4

Commit message: Finished working prototype
Connections:
- net 3.3V: now also U$1.3.3V1
- net 5V: now also IC1P.V+, U$1.5V
- net GND: now also CUSTOM.1, IC1P.V-, U$1.GND2; no longer CUSTOM.2
- net N$17: now also CUSTOM.2; no longer CUSTOM.1
Changed lines of the file:
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@@
 <part name="D5" library="diode" library_urn="urn:adsk.eagle:library:210" deviceset="1N4446" device="" package3d_urn="urn:adsk.eagle:package:43344/2"/>
 <part name="GND8" library="antduino" deviceset="SPARKFUN_GND" device=""/>
+<part name="SUPPLY6" library="SparkFun-PowerSymbols" library_urn="urn:adsk.eagle:library:530" deviceset="5V" device=""/>
+<part name="GND9" library="antduino" deviceset="SPARKFUN_GND" device=""/>
+<part name="P+2" library="antduino" deviceset="SPARKFUN_3.3V" device=""/>
+<part name="GND13" library="antduino" deviceset="SPARKFUN_GND" device=""/>
+<part name="SUPPLY7" library="SparkFun-PowerSymbols" library_urn="urn:adsk.eagle:library:530" deviceset="5V" device=""/>
 </parts>
 <sheets>
@@
 <attribute name="VALUE" x="-80.01" y="28.702" size="1.778" layer="96" rot="R180"/>
 </instance>
-<instance part="CUSTOM" gate="G$1" x="93.98" y="17.78" smashed="yes">
-<attribute name="NAME" x="91.44" y="20.32" size="1.778" layer="95"/>
-<attribute name="VALUE" x="91.44" y="15.24" size="1.778" layer="96"/>
+<instance part="CUSTOM" gate="G$1" x="93.98" y="17.78" smashed="yes" rot="MR0">
+<attribute name="NAME" x="96.52" y="20.32" size="1.778" layer="95" rot="MR0"/>
+<attribute name="VALUE" x="96.52" y="15.24" size="1.778" layer="96" rot="MR0"/>
 </instance>
 <instance part="R11" gate="G$1" x="-55.88" y="33.02" smashed="yes">
@@
 <instance part="GND8" gate="1" x="-121.92" y="121.92" smashed="yes" rot="R180">
 <attribute name="VALUE" x="-119.38" y="124.46" size="1.778" layer="96" rot="R180"/>
+</instance>
+<instance part="SUPPLY6" gate="G$1" x="30.48" y="27.94" smashed="yes" rot="R90">
+<attribute name="VALUE" x="27.686" y="27.94" size="1.778" layer="96" rot="R90" align="bottom-center"/>
+</instance>
+<instance part="GND9" gate="1" x="22.86" y="25.4" smashed="yes" rot="R270">
+<attribute name="VALUE" x="20.32" y="27.94" size="1.778" layer="96" rot="R270"/>
+</instance>
+<instance part="P+2" gate="G$1" x="30.48" y="22.86" smashed="yes" rot="R90">
+<attribute name="VALUE" x="26.924" y="21.844" size="1.778" layer="96" rot="R90"/>
+</instance>
+<instance part="IC1" gate="P" x="170.18" y="7.62" smashed="yes"/>
+<instance part="GND13" gate="1" x="170.18" y="-5.08" smashed="yes">
+<attribute name="VALUE" x="167.64" y="-7.62" size="1.778" layer="96"/>
+</instance>
+<instance part="SUPPLY7" gate="G$1" x="170.18" y="17.78" smashed="yes">
+<attribute name="VALUE" x="170.18" y="20.574" size="1.778" layer="96" align="bottom-center"/>
 </instance>
 </instances>
@@
 <wire x1="99.06" y1="27.94" x2="111.76" y2="27.94" width="0.1524" layer="91"/>
 <wire x1="111.76" y1="27.94" x2="111.76" y2="17.78" width="0.1524" layer="91"/>
-<pinref part="CUSTOM" gate="G$1" pin="2"/>
+<pinref part="CUSTOM" gate="G$1" pin="1"/>
 <wire x1="111.76" y1="17.78" x2="111.76" y2="15.24" width="0.1524" layer="91"/>
 <wire x1="99.06" y1="17.78" x2="111.76" y2="17.78" width="0.1524" layer="91"/>
@@
 <wire x1="-121.92" y1="111.76" x2="-121.92" y2="119.38" width="0.1524" layer="91"/>
 </segment>
+<segment>
+<pinref part="U$1" gate="G$1" pin="GND2"/>
+<pinref part="GND9" gate="1" pin="GND"/>
+<wire x1="35.56" y1="25.4" x2="25.4" y2="25.4" width="0.1524" layer="91"/>
+</segment>
+<segment>
+<pinref part="GND13" gate="1" pin="GND"/>
+<pinref part="IC1" gate="P" pin="V-"/>
+<wire x1="170.18" y1="-2.54" x2="170.18" y2="0" width="0.1524" layer="91"/>
+</segment>
 </net>
 <net name="N$2" class="0">
@@
 <pinref part="P+5" gate="G$1" pin="3.3V"/>
 <wire x1="-5.08" y1="10.16" x2="-5.08" y2="12.7" width="0.1524" layer="91"/>
+</segment>
+<segment>
+<pinref part="U$1" gate="G$1" pin="3.3V1"/>
+<pinref part="P+2" gate="G$1" pin="3.3V"/>
+<wire x1="35.56" y1="22.86" x2="30.48" y2="22.86" width="0.1524" layer="91"/>
 </segment>
 </net>
@@
 <net name="N$17" class="0">
 <segment>
-<pinref part="CUSTOM" gate="G$1" pin="1"/>
-<wire x1="88.9" y1="17.78" x2="88.9" y2="25.4" width="0.1524" layer="91"/>
 <pinref part="U$1" gate="G$1" pin="PC13"/>
 <wire x1="88.9" y1="25.4" x2="76.2" y2="25.4" width="0.1524" layer="91"/>
+<pinref part="CUSTOM" gate="G$1" pin="2"/>
+<wire x1="88.9" y1="25.4" x2="88.9" y2="17.78" width="0.1524" layer="91"/>
 </segment>
 </net>
@@
 <wire x1="-111.76" y1="71.12" x2="-111.76" y2="73.66" width="0.1524" layer="91"/>
 </segment>
-</net>
+<segment>
+<pinref part="U$1" gate="G$1" pin="5V"/>
+<pinref part="SUPPLY6" gate="G$1" pin="5V"/>
+<wire x1="35.56" y1="27.94" x2="30.48" y2="27.94" width="0.1524" layer="91"/>
+</segment>
+<segment>
+<pinref part="SUPPLY7" gate="G$1" pin="5V"/>
+<pinref part="IC1" gate="P" pin="V+"/>
+<wire x1="170.18" y1="17.78" x2="170.18" y2="15.24" width="0.1524" layer="91"/>
+</segment>
+</net>
